File: final_Schematic/final_Schematic.kicad_sch (KiCad schematic)
At the start: 37 parts, among them J1 XT60 (Battery Input), J2 FUSE_2, J3 FUSE _1, K1 SRD-05VDC-SL-C, K2 HEADER_MALE_3X1, K3 TERMINAL_KF235-5.0-3P, K4 TERMINAL_KF235-5.0-3P, K5 SRD-05VDC-SL-C, K6 HEADER_MALE_3X1, Q1 NPN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

Commit message: Schematic_Update_2
Other:
- note added: "6_Channel_Receiver"
Changed lines of the file:
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@@
+		)
+	)
+	(text "6_Channel_Receiver\n"
+		(exclude_from_sim no)
+		(at 114.554 159.766 0)
+		(effects
+			(font
+				(size 1.27 1.27)
+				(color 0 77 0 1)
+			)
 		)
 	)
